File: tbd.sch (KiCad schematic (older format))
At the start: 8 parts, among them J1 USBPCB, P1 CONN_02X04, U1 MKL27ZxxxVFM4

Commit message: Clean up unneeded files, remove v0.1 RTP files since they're in the v0.1 branch
Parts:
- C1, C2: footprint Sparkfun:SparkFun-0402-CAP -> tbd:SparkFun-0402-CAP
- LED1: footprint Sparkfun:SparkFun-LED-0603 -> tbd:SparkFun-LED-0603
- R1, R2: footprint Sparkfun:SparkFun-0402-RES -> tbd:SparkFun-0402-RES
Changed lines of the file:
@@
 LIBS:opto
 LIBS:atmel
-LIBS:SparkFun
 LIBS:contrib
 LIBS:valves
 LIBS:mkl27zxxxvfm4
-LIBS:tbd-cache
+LIBS:tbd
+LIBS:SparkFun
 EELAYER 25 0
 EELAYER END
@@
 F 0 "R2" H 1900 2950 50  0000 L BNN
 F 1 "33R" H 1900 2720 50  0000 L BNN
-F 2 "Sparkfun:SparkFun-0402-RES" H 2300 2650 50  0001 C CNN
+F 2 "tbd:SparkFun-0402-RES" H 2300 2650 50  0001 C CNN
 F 3 "" H 2050 2850 60  0000 C CNN
 	1    2050 2850
@@
 F 0 "R1" H 1900 2850 50  0000 L BNN
 F 1 "33R" H 1900 2620 50  0000 L BNN
-F 2 "Sparkfun:SparkFun-0402-RES" H 2300 2550 50  0001 C CNN
+F 2 "tbd:SparkFun-0402-RES" H 2300 2550 50  0001 C CNN
 F 3 "" H 2050 2750 60  0000 C CNN
 	1    2050 2750
@@
 F 0 "C1" H 2110 3815 50  0000 L BNN
 F 1 "100nF" H 2110 3615 50  0000 L BNN
-F 2 "Sparkfun:SparkFun-0402-CAP" H 2500 3550 50  0001 C CNN
+F 2 "tbd:SparkFun-0402-CAP" H 2500 3550 50  0001 C CNN
 F 3 "" H 2050 3700 60  0000 C CNN
 	1    2050 3700
@@
 F 0 "C2" H 4360 4865 50  0000 L BNN
 F 1 "100nF" H 4360 4665 50  0000 L BNN
-F 2 "Sparkfun:SparkFun-0402-CAP" H 4750 4600 50  0001 C CNN
+F 2 "tbd:SparkFun-0402-CAP" H 4750 4600 50  0001 C CNN
 F 3 "" H 4300 4750 60  0000 C CNN
 	1    4300 4750
@@
 F 0 "LED1" V 2150 2150 50  0000 L BNN
 F 1 "LED0603" V 2550 2150 50  0000 L BNN
-F 2 "Sparkfun:SparkFun-LED-0603" H 2350 2450 50  0001 C CNN
+F 2 "tbd:SparkFun-LED-0603" H 2350 2450 50  0001 C CNN
 F 3 "" H 2350 2300 60  0000 C CNN
 	1    2350 2300

Commit message: Update design to v0.2
Parts:
- added J2: USB-MICROB-5PIN, tbd:SparkFun-USB-MICROB, symbol USB-MICROB-5PIN
- added R1: 100R, Resistors_SMD:R_0603, symbol RESISTOR0402-RES
- added TP1: SWD_CLK, Measurement_Points:Measurement_Point_Round-SMD-Pad_Small, symbol TEST-POINT2
- C1: footprint tbd:SparkFun-0402-CAP -> Capacitors_SMD:C_0603; symbol CAP0603-CAP -> CAP0402-CAP
- C2: footprint tbd:SparkFun-0402-CAP -> Capacitors_SMD:C_0603
- LED1: footprint tbd:SparkFun-LED-0603 -> tbd:LED-0603
- P1: footprint tbd:hdr-boardedge-4x2 -> tbd:HEADER_2x4_SMT_RA
- R2: renamed from R1; footprint tbd:SparkFun-0402-RES -> Resistors_SMD:R_0603; symbol RESISTOR0603-RES -> RESISTOR0402-RES
- R3: renamed from R2; footprint tbd:SparkFun-0402-RES -> Resistors_SMD:R_0603; symbol RESISTOR0603-RES -> RESISTOR0402-RES
Connections:
- net +3.3V: now also P1.1 (P1), R1.1; no longer LED1.A
- net VSS: now also J2.GND, J2.MTN1, J2.MTN2, J2.MTN3, J2.MTN4, J2.MTN5, J2.MTN6; no longer P1.8 (P8)
- net SPI1_SS: now reaches U1.29 (PTD4/LLWU_P14)
- net SPI1_SS: now also P1.2 (P2)
- net SPI1_SCK: now reaches U1.30 (PTD5)
- net SPI1_SCK: now also P1.4 (P4)
- net SPI1_MOSI: now reaches U1.31 (PTD6/LLWU_P15)
- net SPI1_MOSI: now also P1.6 (P6)
- net SPI1_MISO: now reaches U1.32 (PTD7)
- net SPI1_MISO: now also P1.8 (P8)
- net at J1.5V (VBUS), U1.6 (VREGIN): now also J2.VBUS
- net at J1.DN (D-), R3.1: now also J2.D-
- net at J1.DP (D+), R2.1: now also J2.D+
- net /NMI renamed I2C1_SDA
- net I2C1_SDA: now also P1.3 (P3); no longer P1.6 (P6)
- net /RESET: no longer names the net of U1.19 (PTA20)
- net /RESET: no longer P1.5 (P5)
- net LPUART0_RX: no longer names the net of U1.11 (PTA1)
- net LPUART0_RX: no longer P1.1 (P1)
- net LPUART0_TX: no longer names the net of U1.12 (PTA2)
- net LPUART0_TX: no longer P1.3 (P3)
- net SWD_CLK: no longer names the net of U1.10 (PTA0)
- net SWD_CLK: now also TP1.1; no longer P1.2 (P2)
- net SWD_DIO renamed I2C1_SCL
- net I2C1_SCL: now also P1.5 (P5); no longer P1.4 (P4)
- new net: LED1.A, R1.2
Other:
- moved on the sheet: J1, LED1
